File: pcb/avr-sensors.sch (KiCad schematic (older format))
At the start: 41 parts, among them CON1 BARREL_JACK, IC1 REG1117, IC2 ATMEGA328P-A, J1 BUS, J2 GPIO, J3 ICSP, J4 PWR-1W, J5 PWR-DHT, J6 IO, J7 OLED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

Commit message: pcb: Fixed wrong value of the Ethernet termination resistors
Value was 49k9, corrected to 49.9
Parts:
- R7, R8: value 49k9 1% -> 49.9 1%
Changed lines of the file:
@@
 LIBS:J0026D21BNL
 LIBS:avr-sensors-cache
-EELAYER 27 0
+EELAYER 24 0
 EELAYER END
 $Descr A4 11693 8268
@@
 P 8600 4400
 F 0 "R7" V 8680 4400 40  0000 C CNN
-F 1 "49k9 1%" V 8607 4401 40  0000 C CNN
+F 1 "49.9 1%" V 8607 4401 40  0000 C CNN
 F 2 "~" V 8530 4400 30  0000 C CNN
 F 3 "~" H 8600 4400 30  0000 C CNN
@@
 P 8600 5000
 F 0 "R8" V 8680 5000 40  0000 C CNN
-F 1 "49k9 1%" V 8607 5001 40  0000 C CNN
+F 1 "49.9 1%" V 8607 5001 40  0000 C CNN
 F 2 "~" V 8530 5000 30  0000 C CNN
 F 3 "~" H 8600 5000 30  0000 C CNN

Commit message: pcb: Changed wrong resistor value
Value of the Ethernet termination resistors used was 49k9 instead of 49.9.
Parts:
- R5, R6: value 49k9 1% -> 49.9 1%
Changed lines of the file:
@@
 P 8600 3050
 F 0 "R5" V 8680 3050 40  0000 C CNN
-F 1 "49k9 1%" V 8607 3051 40  0000 C CNN
+F 1 "49.9 1%" V 8607 3051 40  0000 C CNN
 F 2 "~" V 8530 3050 30  0000 C CNN
 F 3 "~" H 8600 3050 30  0000 C CNN
@@
 P 8600 3650
 F 0 "R6" V 8680 3650 40  0000 C CNN
-F 1 "49k9 1%" V 8607 3651 40  0000 C CNN
+F 1 "49.9 1%" V 8607 3651 40  0000 C CNN
 F 2 "~" V 8530 3650 30  0000 C CNN
 F 3 "~" H 8600 3650 30  0000 C CNN

Commit message: pcb: Changed the value of crystal capacitors to 22pF
Changed the previously undefined value of the two capacitors connected to the
25MHz crystal to 22pF.
Parts:
- C8, C9: value C -> 22pF
Changed lines of the file:
@@
 P 7650 6550
 F 0 "C8" H 7650 6650 40  0000 L CNN
-F 1 "C" H 7656 6465 40  0000 L CNN
+F 1 "22pF" H 7656 6465 40  0000 L CNN
 F 2 "~" H 7688 6400 30  0000 C CNN
 F 3 "~" H 7650 6550 60  0000 C CNN
@@
 P 8250 6550
 F 0 "C9" H 8250 6650 40  0000 L CNN
-F 1 "C" H 8256 6465 40  0000 L CNN
+F 1 "22pF" H 8256 6465 40  0000 L CNN
 F 2 "~" H 8288 6400 30  0000 C CNN
 F 3 "~" H 8250 6550 60  0000 C CNN
